File: KiCad/anorith.kicad_pcb (KiCad board)
At the start: 4 copper layers, 65 x 30 mm, 45 parts, among them J1 Conn_02x20_Counter_Clockwise, J3 USB_C_Receptacle_USB2.0_14P, SW1 RESET, SW2 BOOT, U1 RP2040, U2 AMS1117-3.3, U3 W25Q16JVSS, Y1 12MHz

Commit message: prod
Parts:
- added dialgorithm: dialgorithm, dialgorithm:dialgorithm, F.Cu at (174.5, 107.2)
- added dialgorithm: dialgorithm, dialgorithm:dialgorithm, B.Cu at (174.9, 107.2)

Commit message: Update anorith.kicad_pcb
Parts:
- removed SW1: RESET, Button_Switch_THT:SW_PUSH_6mm
- removed SW2: BOOT, Button_Switch_THT:SW_PUSH_6mm
